Commit message: add amcl

File: catkin_ws/src/my_robot/urdf/my_robot.xacro (robot description, xacro)
@@ -184,3 +184,11 @@
     <axis xyz="0 1 0" rpy="0 0 0"/>
   </joint>
+  <!-- Stereo camera -->
+  <joint name="camera_optical_joint" type="fixed">
+    <origin xyz="0 0 0" rpy="-1.5707 0 -1.5707"/>
+    <parent link="camera"/>
+    <child link="camera_link_optical"/>
+  </joint>
+  <link name="camera_link_optical">
+  </link>
 </robot>
